Commit message: zmiana nazwy package, udpate readme

File: urdf/IRB7600v2.urdf (robot description, URDF)
Before this commit: robot IRB7600, 8 links, 7 joints
Links:
- removed link effector
- added link tool; visual cylinder length=0.01 radius=0.2
Joints:
- removed joint base_to_right_link1
- removed joint link6_effector
- added joint base_link_link1: type continuous, parent base_link, child link1, origin xyz=0 0 0.78 rpy=0 0 0, axis 0 0 1
- added joint link6_tool: type fixed, parent link6, child tool, origin xyz=0 0 0.25 rpy=0 0 0
- joint link1_link2: origin xyz=0.41 0 0.78 rpy=1.571 0 0 -> xyz=0.41 0 0 rpy=1.571 -1.571 0
- joint link2_link3: origin xyz=0 1.075 0 rpy=0 0 1.571 -> xyz=1.075 0 0 rpy=0 0 0
- joint link3_link4: origin xyz=0.165 0 0 rpy=1.571 0 0 -> xyz=0.165 -1.056 0 rpy=1.571 0 0
- joint link4_link5: origin xyz=0 0 1.056 rpy=-1.571 0 0 -> xyz=0 0 0 rpy=-1.571 0 0
